File: BuildUpons-CenterLED.brd (EAGLE design)
At the start: 3.5 x 6.5 mm, 4 parts, among them J1 METAL-LEGMOREPASTE, J2 METAL-LEGMOREPASTE

Commit message: FR4 Jig cut complete
Parts:
- moved D1 0.40 mm to (0.00, 0.00)
